File: schiffre_pico/schiffre_pico.kicad_sch (KiCad schematic)
At the start: 6 parts, among them U5 Pico

Commit message: small drc things
Connections:
- net GND: now also U5.13 (GND); no longer U5.35 (ADC_VREF)
- no-connect marks 4 -> 7
